Commit message: Update stochlite.urdf

File: urdf/stochlite.urdf (robot description, URDF)
Before this commit: robot stochlite, 24 links, 23 joints
Links:
- added link bl_leg_frame
- added link br_leg_frame
- added link fl_leg_frame
- added link fr_leg_frame
Joints:
- added joint bl_fixed: type fixed, parent base_link, child bl_leg_frame, origin xyz=-0.16695 0.0956 -0.0049999 rpy=0 0 0, axis 1 0 0
- added joint br_fixed: type fixed, parent base_link, child br_leg_frame, origin xyz=-0.16695 -0.0964 -0.0050001 rpy=0 0 0, axis 1 0 0
- added joint fl_fixed: type fixed, parent base_link, child fl_leg_frame, origin xyz=0.16695 0.0956 -0.0050001 rpy=0 0 0, axis 1 0 0
- added joint fr_fixed: type fixed, parent base_link, child fr_leg_frame, origin xyz=0.16695 -0.0964 -0.0049999 rpy=0 0 0, axis 1 0 0
