Commit message: Update stochlite.description.xacro

File: urdf/stochlite.description.xacro (robot description, xacro)
@@ -7,12 +7,14 @@
     <xacro:property name="hip_lim" value="10.22" />
     <xacro:property name="knee_lim" value="10.22" />
-    <xacro:macro name="stochlite_description">
+    <xacro:macro name="stochlite_description" params="fixed">
         <!-- For KDL -->
-        <!-- <link name="dummy">
-        </link>
-        <joint name="dummy_joint" type="fixed">
-            <parent link="dummy"/>
-            <child link="base_link"/>
-        </joint> -->
+        <xacro:if value="${fixed}">
+            <link name="world">
+            </link>
+            <joint name="fixed" type="fixed">
+                <parent link="world"/>
+                <child link="base_link"/>
+            </joint>
+        </xacro:if>
         <link name="base_link">
             <inertial>

Commit message: Update

File: urdf/stochlite.description.xacro (robot description, xacro)
@@ -4,5 +4,5 @@
     <xacro:property name="torque" value="4.1" />
     <xacro:property name="velocity" value="4.6" />
-    <xacro:property name="abd_lim" value="1.572" />
+    <xacro:property name="abd_lim" value="10.22" />
     <xacro:property name="hip_lim" value="10.22" />
     <xacro:property name="knee_lim" value="10.22" />
@@ -17,4 +17,12 @@
             </joint>
         </xacro:if>
+        <xacro:unless value="${fixed}">
+            <link name="dummy">
+            </link>
+            <joint name="dummy_joint" type="fixed">
+                <parent link="dummy"/>
+                <child link="base_link"/>
+            </joint>
+        </xacro:unless>
         <link name="base_link">
             <inertial>

File: urdf/stochlite.gazebo.xacro (robot description, xacro)
@@ -8,7 +8,7 @@
             </plugin>
         </gazebo>
-        <!-- <gazebo>
+        <gazebo>
             <self_collide>1</self_collide>
-        </gazebo> -->
+        </gazebo>
         <gazebo>
             <plugin filename="libgazebo_ros_p3d.so" name="p3d_base_controller">

File: urdf/stochlite.sensors.xacro (robot description, xacro)
@@ -27,5 +27,5 @@
                 <updateRate>${update_rate}</updateRate>
                 <bodyName>imu_link_${id}</bodyName>
-                <topicName>imu_${id}/data</topicName>
+                <topicName>sensors/imu_${id}</topicName>
                 <accelDrift>0.005 0.005 0.005</accelDrift>
                 <accelGaussianNoise>${gnoise} ${gnoise} ${gnoise}</accelGaussianNoise>
@@ -89,5 +89,5 @@
                 </ray>
                 <plugin name="tof_plugin_${id}" filename="libgazebo_ros_range.so">
-                    <topicName>gazebo/range_tof_${id}</topicName>
+                    <topicName>sensors/range_tof_${id}</topicName>
                     <frameName>frame_range_tof_${id}</frameName>
                     <gaussianNoise>${gnoise}</gaussianNoise>
@@ -100,3 +100,17 @@
         </gazebo>
     </xacro:macro>
+    <!-- Contact Sensor Plugins -->
+    <xacro:macro name="contact_sensor" params="leg_name">
+        <gazebo reference="${leg_name}_shank_link">
+            <sensor name="${leg_name}_link_contact_sensor" type="contact">
+                <contact>
+                    <collision>${leg_name}_shank_link_collision</collision>
+                </contact>
+                <plugin name="gazebo_ros_bumper_controller" filename="libgazebo_ros_bumper.so">
+                    <bumperTopicName>${leg_name}_contact</bumperTopicName>
+                    <frameName>${leg_name}_shank_link</frameName>
+                </plugin>
+            </sensor>
+        </gazebo>
+    </xacro:macro>
 </robot>

File: urdf/stochlite.urdf (robot description, URDF)
Before this commit: robot stochlite, 28 links, 27 joints
Links:
- added link dummy
Joints:
- added joint dummy_joint: type fixed, parent dummy, child base_link
- joint bl_abd_joint: limit lower=-1.572 upper=1.572 effort=4.1 velocity=4.6 -> lower=-10.22 upper=10.22 effort=4.1 velocity=4.6
- joint br_abd_joint: limit lower=-1.572 upper=1.572 effort=4.1 velocity=4.6 -> lower=-10.22 upper=10.22 effort=4.1 velocity=4.6
- joint fl_abd_joint: limit lower=-1.572 upper=1.572 effort=4.1 velocity=4.6 -> lower=-10.22 upper=10.22 effort=4.1 velocity=4.6
- joint fr_abd_joint: limit lower=-1.572 upper=1.572 effort=4.1 velocity=4.6 -> lower=-10.22 upper=10.22 effort=4.1 velocity=4.6

File: urdf/stochlite.urdf.xacro (robot description, xacro)
@@ -40,12 +40,16 @@
     <xacro:stochlite_gazebo />
     <!-- For sensors-->
-    <xacro:imu id="1" x="0.0" y="0.0" z="0.005" roll="0.0" pitch="0.0" yaw="0.0" update_rate="20" gnoise="0.005"/>
+    <xacro:imu id="1" x="0.0" y="0.0" z="0.005" roll="0.0" pitch="0.0" yaw="0.0" update_rate="100" gnoise="0.005"/>
     <!-- front triangle of tofs -->
-    <xacro:tof id="1" x="0.150" y=" 0.000" z="-0.025" roll="0.0" pitch="1.57" yaw="0.0" update_rate="20" gnoise="0.0001"/>
-    <xacro:tof id="2" x="0.065" y=" 0.047" z="-0.025" roll="0.0" pitch="1.57" yaw="0.0" update_rate="20" gnoise="0.0001"/>
-    <xacro:tof id="6" x="0.065" y="-0.047" z="-0.025" roll="0.0" pitch="1.57" yaw="0.0" update_rate="20" gnoise="0.0001"/>
+    <xacro:tof id="1" x="0.150" y=" 0.000" z="-0.025" roll="0.0" pitch="1.57" yaw="0.0" update_rate="20" gnoise="0.005"/>
+    <xacro:tof id="2" x="0.065" y=" 0.047" z="-0.025" roll="0.0" pitch="1.57" yaw="0.0" update_rate="20" gnoise="0.005"/>
+    <xacro:tof id="6" x="0.065" y="-0.047" z="-0.025" roll="0.0" pitch="1.57" yaw="0.0" update_rate="20" gnoise="0.005"/>
     <!-- back triangle of tofs -->
-    <xacro:tof id="4" x="-0.150" y=" 0.000" z="-0.025" roll="0.0" pitch="1.57" yaw="0.0" update_rate="20" gnoise="0.0001"/>
-    <xacro:tof id="3" x="-0.065" y=" 0.047" z="-0.025" roll="0.0" pitch="1.57" yaw="0.0" update_rate="20" gnoise="0.0001"/>
-    <xacro:tof id="5" x="-0.065" y="-0.047" z="-0.025" roll="0.0" pitch="1.57" yaw="0.0" update_rate="20" gnoise="0.0001"/>
+    <xacro:tof id="4" x="-0.150" y=" 0.000" z="-0.025" roll="0.0" pitch="1.57" yaw="0.0" update_rate="20" gnoise="0.005"/>
+    <xacro:tof id="3" x="-0.065" y=" 0.047" z="-0.025" roll="0.0" pitch="1.57" yaw="0.0" update_rate="20" gnoise="0.005"/>
+    <xacro:tof id="5" x="-0.065" y="-0.047" z="-0.025" roll="0.0" pitch="1.57" yaw="0.0" update_rate="20" gnoise="0.005"/>
+    <xacro:contact_sensor leg_name="fl"/>
+    <xacro:contact_sensor leg_name="fr"/>
+    <xacro:contact_sensor leg_name="bl"/>
+    <xacro:contact_sensor leg_name="br"/>
 </robot>

File: urdf/stochlite_fixed.urdf (robot description, URDF)
Before this commit: robot stochlite, 29 links, 28 joints
Joints:
- joint bl_abd_joint: limit lower=-1.572 upper=1.572 effort=4.1 velocity=4.6 -> lower=-10.22 upper=10.22 effort=4.1 velocity=4.6
- joint br_abd_joint: limit lower=-1.572 upper=1.572 effort=4.1 velocity=4.6 -> lower=-10.22 upper=10.22 effort=4.1 velocity=4.6
- joint fl_abd_joint: limit lower=-1.572 upper=1.572 effort=4.1 velocity=4.6 -> lower=-10.22 upper=10.22 effort=4.1 velocity=4.6
- joint fr_abd_joint: limit lower=-1.572 upper=1.572 effort=4.1 velocity=4.6 -> lower=-10.22 upper=10.22 effort=4.1 velocity=4.6
